Commit message: Sync tested robot code and remove generated build files

File: 源码（国赛）/src/yzbot/mybot_description/urdf/arm.xacro (robot description, xacro)
@@ -93,5 +93,5 @@
         <origin xyz="0 0 ${base_h / 2 + link1_len / 2}" rpy="0 0 0" />
         <axis xyz="0 0 1" />
-        <limit lower="-3.14" upper="3.14" effort="300" velocity="1.0" />
+        <limit lower="-3.14" upper="3.14" effort="300" velocity="2.0" />
         <joint_properties damping="50" friction="1" />
     </joint>
@@ -136,5 +136,5 @@
         <origin xyz="0 0 ${link1_len/2}" rpy="0 0 0" />
         <axis xyz="0 1 0" />
-        <limit effort="300" velocity="1.0" lower="-2.35" upper="2.35" />
+        <limit effort="300" velocity="2.0" lower="-2.35" upper="2.35" />
         <joint_properties damping="50" friction="1" />
     </joint>
@@ -163,5 +163,5 @@
         <origin xyz="0 0 ${link2_len}" rpy="0 0 0" />
         <axis xyz="0 1 0" />
-        <limit effort="300" velocity="1.0" lower="-2.62" upper="2.62" />
+        <limit effort="300" velocity="2.0" lower="-2.62" upper="2.62" />
         <joint_properties damping="50" friction="1" />
     </joint>
@@ -190,5 +190,5 @@
         <origin xyz="0 0 ${link3_len}" rpy="0 0 0" />
         <axis xyz="0 0 1" />
-        <limit lower="-3.14" upper="3.14" effort="300" velocity="1.0" />
+        <limit lower="-3.14" upper="3.14" effort="300" velocity="2.0" />
         <joint_properties damping="50" friction="1" />
     </joint>
@@ -217,5 +217,5 @@
         <origin xyz="0 0 ${link4_len}" rpy="0 0 0" />
         <axis xyz="0 -1 0" />
-        <limit effort="300" velocity="1.0" lower="-2.04" upper="2.04" />
+        <limit effort="300" velocity="2.0" lower="-2.04" upper="2.04" />
         <joint_properties damping="50" friction="1" />
     </joint>
@@ -244,5 +244,5 @@
         <origin xyz="0 0 ${link5_len}" rpy="0 0 0" />
         <axis xyz="0 0 1" />
-        <limit lower="-3.14" upper="3.14" effort="300" velocity="1.0" />
+        <limit lower="-3.14" upper="3.14" effort="300" velocity="2.0" />
         <joint_properties damping="50" friction="1" />
     </joint>
@@ -273,5 +273,5 @@
             rpy="0 ${M_PI/2} 0" />
         <axis xyz="0 1 0" />
-        <limit effort="100" lower="0" upper="${link6_rad+gripper_w}" velocity="1.0" />
+        <limit effort="100" lower="0" upper="${link6_rad+gripper_w}" velocity="2.0" />
         <dynamics damping="50" friction="1" />
     </joint>

File: 源码（国赛）/src/yzbot/mybot_description/urdf/originbot_with_arm_gazebo.xacro (robot description, xacro)
@@ -134,5 +134,5 @@
             <!-- limits -->
             <max_wheel_torque>5</max_wheel_torque>
-            <max_wheel_acceleration>0.5</max_wheel_acceleration>
+            <max_wheel_acceleration>5.0</max_wheel_acceleration>
             <!-- output -->
             <command_topic>cmd_vel</command_topic>
