Commit message: feat(robot): add round omni chassis and predictive navigation
Integrate a circular four-omni-wheel chassis, independent arm pedestal
alignment, dual side lidars, and selectable Gazebo/MoveIt/Nav2 profiles.
Add known obstacle trajectory prediction, ordered path tracking, and
fine low-speed sampling to avoid doorway corner cutting and stalls.
Set the new profile to 4 m/s with stronger acceleration and braking,
while retaining collision, prediction, and stale-data protections.

Record three reset five-cube tasks at 195.0, 207.5, and 190.9 simulation
seconds (197.8 s mean), with all 15 placements inside their target zones.
Include model sources, exported meshes, validation tools, and evidence.
The ideal Gazebo planar driver does not establish physical traction or
braking performance; no matched full-task legacy-speed comparison exists.

File: src/yzbot/mybot_description/urdf/lidar_gazebo.xacro (robot description, xacro)
@@ -2,5 +2,5 @@
 <robot xmlns:xacro="http://www.ros.org/wiki/xacro" name="laser">
     <xacro:macro name="lidar"
-        params="prefix:=laser gz_visualize:=false range_min:=0.10 range_max:=30.0 topic:=scan show_visual:=true">
+        params="prefix:=laser gz_visualize:=false range_min:=0.10 range_max:=30.0 topic:=scan show_visual:=true samples:=1441 update_rate:=10 min_angle:=-3.14159 max_angle:=3.14159">
         <!-- Create laser reference frame -->
         <link name="${prefix}_link">
@@ -10,4 +10,9 @@
                 <inertia ixx="0.01" ixy="0.0" ixz="0.0" iyy="0.01" iyz="0.0" izz="0.01" />
             </inertial>
+            <xacro:if value="${prefix == 'laser_left' or prefix == 'laser_right'}">
+            <xacro:mecanum_visual link="${prefix}_link"/>
+            <collision name="mecanum_scanner_housing"><geometry><cylinder radius="0.0355" length="0.034"/></geometry></collision>
+            <collision name="mecanum_scanner_bracket"><origin xyz="-0.025 0 -0.025"/><geometry><box size="0.12 0.086 0.008"/></geometry></collision>
+            </xacro:if>
             <xacro:if value="${show_visual}"><visual>
                 <origin xyz=" 0 0 0 " rpy="0 0 0" />
@@ -32,16 +37,16 @@
         <gazebo reference="${prefix}_link">
             <sensor type="ray" name="${prefix}_lidar">
-                <update_rate>10</update_rate>
+                <update_rate>${update_rate}</update_rate>
                 <visualize>${gz_visualize}</visualize>
                 <ray>
                     <scan>
                         <horizontal>
-                            <!-- 0.25 degree rays: at 7 m their 3.1 cm spacing
-                                 stays below the 5 cm costmap cell size. -->
-                            <samples>1441</samples>
+                            <!-- Defaults use 0.25 degree rays. The round dual
+                                 lidar model uses 0.333 degree rays (4.1 cm at 7 m). -->
+                            <samples>${samples}</samples>
                             <!-- One returned range per ray: interpolation creates phantom edge hits. -->
                             <resolution>1</resolution>
-                            <min_angle>-3.14159</min_angle>
-                            <max_angle>3.14159</max_angle>
+                            <min_angle>${min_angle}</min_angle>
+                            <max_angle>${max_angle}</max_angle>
                         </horizontal>
                     </scan>
