Commit message: feat(sim): adopt validated body-force drive and motion limits
Add a bounded body velocity servo with passive wheels and physical wrench
telemetry. Keep wheel and body-force drivers mutually exclusive.

Configure the office scene for 6 m/s and 4 rad/s, linear and angular
acceleration/braking of 10, and forward/lateral/yaw caps of 1000.
Synchronize predictive motion limits, scene generation and drive defaults.

Include native sampling, repeated headless flow runners, route/force plots
and diagnostic records, retaining failed and interrupted attempts.

Validation: 15-package build, 49 Python tests, C++ tests with no failures,
and one headless five-item flow with valid final positions/heights and no
collision or instability abort. Task time: 120.75 wall / 115.3 sim seconds.

File: src/yzbot/mybot_description/urdf/originbot_with_arm_gazebo.xacro (robot description, xacro)
@@ -120,4 +120,7 @@
     <xacro:wheel_transmission prefix="left" />
     <xacro:wheel_transmission prefix="right" />
+    <!-- Select one actuator only; default on the research branch is body force. -->
+    <xacro:property name="drive_model" value="$(optenv AIC_DRIVE_MODEL body_force)" />
+    <xacro:if value="${dict(wheel=True, body_force=False)[drive_model]}">
     <gazebo>
         <plugin name="differential_drive_controller" filename="libgazebo_ros_diff_drive.so">
@@ -143,3 +146,20 @@
         </plugin>
     </gazebo>
+    </xacro:if>
+    <xacro:if value="${dict(wheel=False, body_force=True)[drive_model]}">
+      <gazebo>
+        <plugin name="body_force_controller" filename="libaic_body_drive.so">
+          <body_link>base_footprint</body_link>
+          <publish_rate>30</publish_rate>
+          <command_timeout>0.5</command_timeout>
+          <max_linear_speed>$(optenv AIC_BODY_MAX_LINEAR_SPEED 6.0)</max_linear_speed>
+          <max_angular_speed>$(optenv AIC_BODY_MAX_ANGULAR_SPEED 4.0)</max_angular_speed>
+          <forward_kp>300</forward_kp><forward_ki>150</forward_ki><forward_limit>1000</forward_limit>
+          <lateral_kp>1000</lateral_kp><lateral_ki>300</lateral_ki><lateral_limit>1000</lateral_limit>
+          <yaw_kp>200</yaw_kp><yaw_ki>100</yaw_ki><yaw_limit>1000</yaw_limit>
+          <odometry_frame>odom</odometry_frame>
+          <robot_base_frame>base_footprint</robot_base_frame>
+        </plugin>
+      </gazebo>
+    </xacro:if>
 </robot>
